Commit message: added basic simulated pick and place funtionality

File: urdf/ur5e_joint_limited_robotiq_2f_85.urdf.xacro (robot description, xacro)
@@ -2,26 +2,15 @@
 <robot xmlns:xacro="http://ros.org/wiki/xacro"
        name="ur5e" >
+  <xacro:property name="prefix" value=""/>
   <!-- common stuff -->
   <xacro:include filename="$(find ur_e_description)/urdf/common.gazebo.xacro" />
   <!-- ur5e -->
-  <xacro:include filename="$(find ur_e_description)/urdf/ur5e.urdf.xacro" />
+  <xacro:include filename="$(find ur5e_workstation)/urdf/ur5e.urdf.xacro" />
   <!-- updated robotiq_2f_85 gripper -->
   <xacro:include filename="$(find robotiq_2f_85_full)/urdf/robotiq_2f_85_full.urdf.xacro" />
   <!-- arm -->
-  <xacro:ur5e_robot prefix="" joint_limited="true"
-    shoulder_pan_lower_limit="${-pi}" shoulder_pan_upper_limit="${pi}"
-    shoulder_lift_lower_limit="${-pi}" shoulder_lift_upper_limit="${pi}"
-    elbow_joint_lower_limit="${-pi}" elbow_joint_upper_limit="${pi}"
-    wrist_1_lower_limit="${-2*pi}" wrist_1_upper_limit="${2*pi}"
-    wrist_2_lower_limit="${-2*pi}" wrist_2_upper_limit="${2*pi}"
-    wrist_3_lower_limit="${-2*pi}" wrist_3_upper_limit="${2*pi}"
-  />
+  <xacro:ur5e prefix="" joint_limited="false"/>
   <!-- gripper -->
   <xacro:robotiq_2f_85_full prefix=""/>
-  <joint name="robotiq_85_adapters_joint" type="fixed">
-    <parent link="tool0"/>
-    <child link="realsense_camera_mount_link"/>
-    <origin xyz="0.0235 -0.0535 0.0115" rpy="1.5707 0.0 -0.785" />
-  </joint>
   <!-- world -->
   <link name="world" />
@@ -32,3 +21,8 @@
     <origin xyz="0.0 0.0 0.0" rpy="0.0 0.0 0.0" />
   </joint>
+  <joint name="${prefix}robotiq_85_adapters_joint" type="fixed">
+    <parent link="${prefix}tool0"/>
+    <child link="${prefix}realsense_camera_mount_link"/>
+    <origin xyz="0.0235 -0.0535 0.0115" rpy="1.5707 0.0 -0.785" />
+  </joint>
 </robot>
