Commit message: adding/testing new configurations

File: urdf/ur5e_D435_robotiq_2f.urdf (robot description, URDF)
Before this commit: robot ur5e, 20 links, 19 joints
Joints:
- joint robotiq_2f_85_body_to_robotiq_2f_85_left_finger_joint: type fixed -> passive
- joint robotiq_2f_85_body_to_robotiq_2f_85_right_finger_joint: type fixed -> passive
