Commit message: updated new config for ur5e with robotiq 2f 85 gripper: wrong mounting orientation

File: urdf/ur5e_r85.urdf.xacro (robot description, xacro)
@@ -28,5 +28,5 @@
     <parent link="tool0" />
     <child link = "wrist_adapter_link" />
-    <origin xyz="0.0 0.0 0.0" rpy="0.0 0.0 0.0" />
+    <origin xyz="0.0 0.0 0.1" rpy="0.0 0.0 0.0" />
   </joint>
   <xacro:robotiq_arg2f_85 prefix="gripper_"/>
@@ -34,5 +34,5 @@
     <parent link="wrist_adapter_link"/>
     <child link="gripper_robotiq_arg2f_base_link"/>
-    <origin xyz="0.0 0.0 0.0" rpy="0.0 0.0 0.0" />
+    <origin xyz="0.0 0.0 0.1" rpy="0.0 0.0 0.0" />
   </joint>
 </robot>
