Commit message: urdf: mounts combined w ur5e

File: urdf/ur5e.urdf.xacro (robot description, xacro)
@@ -350,4 +350,11 @@
       <child link="${prefix}tool0"/>
     </joint>
+    <!-- Artificial end link (TCP) -->
+    <link name="${prefix}virtual_tcp_link"/>
+    <joint name="${prefix}tool0-virtual_tcp_link_joint" type="fixed">
+      <origin xyz="0 0 0.21" rpy="0 0 0"/>
+      <parent link="${prefix}tool0"/>
+      <child link="${prefix}virtual_tcp_link"/>
+    </joint>
   </xacro:macro>
 </robot>
