Commit message: add: urdf files - moved for sim convenience, revised: gazebo controler/transmission .yaml files

File: urdf/ur5e_with_r85_mounting_structure.urdf.xacro (robot description, xacro)
@@ -1,4 +1,16 @@
 <?xml version="1.0"?>
-<robot xmlns:xacro="http://ros.org/wiki/xacro">
+<robot xmlns:xi="http://www.w3.org/2001/XInclude"
+    xmlns:gazebo="http://playerstage.sourceforge.net/gazebo/xmlschema/#gz"
+    xmlns:model="http://playerstage.sourceforge.net/gazebo/xmlschema/#model"
+    xmlns:sensor="http://playerstage.sourceforge.net/gazebo/xmlschema/#sensor"
+    xmlns:body="http://playerstage.sourceforge.net/gazebo/xmlschema/#body"
+    xmlns:geom="http://playerstage.sourceforge.net/gazebo/xmlschema/#geom"
+    xmlns:joint="http://playerstage.sourceforge.net/gazebo/xmlschema/#joint"
+    xmlns:controller="http://playerstage.sourceforge.net/gazebo/xmlschema/#controller"
+    xmlns:interface="http://playerstage.sourceforge.net/gazebo/xmlschema/#interface"
+    xmlns:rendering="http://playerstage.sourceforge.net/gazebo/xmlschema/#rendering"
+    xmlns:renderable="http://playerstage.sourceforge.net/gazebo/xmlschema/#renderable"
+    xmlns:physics="http://playerstage.sourceforge.net/gazebo/xmlschema/#physics"
+    xmlns:xacro="http://ros.org/wiki/xacro" name="ur5e" >
   <xacro:macro name="cylinder_inertial" params="radius length mass *origin">
     <inertial>
@@ -20,6 +32,8 @@
     safety_limits:=false safety_pos_margin:=0.15
     safety_k_position:=20">
-    <xacro:include filename="$(find ur_e_description)/urdf/ur.transmission.xacro" />
-    <xacro:include filename="$(find ur_e_description)/urdf/ur.gazebo.xacro" />
+    <xacro:include filename="$(find ur5e_workstation)/urdf/ur_e_transmission.xacro" />
+    <xacro:include filename="$(find ur5e_workstation)/urdf/ur_e_gazebo.xacro" />
+    <xacro:ur_arm_transmission prefix="${prefix}" />
+    <xacro:ur_arm_gazebo prefix="${prefix}" />
     <!-- Inertia parameters -->
     <xacro:property name="base_mass" value="4.0" />  <!-- This mass might be incorrect -->
@@ -112,5 +126,5 @@
         </xacro:if>
       </xacro:if>
-      <dynamics damping="0.0" friction="0.0"/>
+      <dynamics damping="0.7" friction="0.0"/>
     </joint>
     <link name="${prefix}shoulder_link">
@@ -149,5 +163,5 @@
         </xacro:if>
       </xacro:if>
-      <dynamics damping="0.0" friction="0.0"/>
+      <dynamics damping="0.7" friction="0.0"/>
     </joint>
     <link name="${prefix}upper_arm_link">
@@ -186,5 +200,5 @@
         </xacro:if>
       </xacro:if>
-      <dynamics damping="0.0" friction="0.0"/>
+      <dynamics damping="0.7" friction="0.0"/>
     </joint>
     <link name="${prefix}forearm_link">
@@ -223,5 +237,5 @@
         </xacro:if>
       </xacro:if>
-      <dynamics damping="0.0" friction="0.0"/>
+      <dynamics damping="0.7" friction="0.0"/>
     </joint>
     <link name="${prefix}wrist_1_link">
@@ -260,5 +274,5 @@
         </xacro:if>
       </xacro:if>
-      <dynamics damping="0.0" friction="0.0"/>
+      <dynamics damping="0.7" friction="0.0"/>
     </joint>
     <link name="${prefix}wrist_2_link">
@@ -297,5 +311,5 @@
         </xacro:if>
       </xacro:if>
-      <dynamics damping="0.0" friction="0.0"/>
+      <dynamics damping="0.7" friction="0.0"/>
     </joint>
     <link name="${prefix}wrist_3_link">
@@ -330,6 +344,4 @@
       </collision>
     </link>
-    <xacro:ur_arm_transmission prefix="${prefix}" />
-    <xacro:ur_arm_gazebo prefix="${prefix}" />
     <!-- ROS base_link to UR 'Base' Coordinates transform -->
     <link name="${prefix}base"/>

File: urdf/ur_e_gazebo.xacro (robot description, xacro)
@@ -13,18 +13,26 @@
     xmlns:physics="http://playerstage.sourceforge.net/gazebo/xmlschema/#physics"
     xmlns:xacro="http://ros.org/wiki/xacro" name="ur5e_d435_millibar_combined_r2f85" >
-  <xacro:include filename="$(find ur5e_workstation)/urdf/ur5e_with_r85_mounting_structure.urdf.xacro" />
-  <xacro:include filename="$(find robotiq_2f_85_gripper_visualization)/urdf/robotiq_arg2f_85_model_macro.xacro" />
-  <xacro:ur5e prefix="robot_" joint_limited="false"/>
-  <link name="world" />
-  <joint name="world_joint" type="fixed">
-    <parent link="world" />
-    <child link = "robot_base_link" />
-    <origin xyz="0.0 0.0 0.0" rpy="0.0 0.0 0.0" />
-  </joint>
-  <xacro:robotiq_arg2f_85 prefix="gripper_"/>
-  <joint name="robotiq_2f_85_connector_joint" type="fixed">
-    <parent link="robot_r85_network_adapter_link"/>
-    <child link="gripper_robotiq_arg2f_base_link"/>
-    <origin xyz="0.0 0.0 0.005" rpy="0.0 0.0 -1.57" />
-  </joint>
+  <xacro:macro name="ur_arm_gazebo" params="prefix">
+    <gazebo reference="${prefix}shoulder_link">
+      <selfCollide>true</selfCollide>
+    </gazebo>
+    <gazebo reference="${prefix}upper_arm_link">
+      <selfCollide>true</selfCollide>
+    </gazebo>
+    <gazebo reference="${prefix}forearm_link">
+      <selfCollide>true</selfCollide>
+    </gazebo>
+    <gazebo reference="${prefix}wrist_1_link">
+      <selfCollide>true</selfCollide>
+    </gazebo>
+    <gazebo reference="${prefix}wrist_3_link">
+      <selfCollide>true</selfCollide>
+    </gazebo>
+    <gazebo reference="${prefix}wrist_2_link">
+      <selfCollide>true</selfCollide>
+    </gazebo>
+    <gazebo reference="${prefix}ee_link">
+      <selfCollide>true</selfCollide>
+    </gazebo>
+  </xacro:macro>
 </robot>

Commit message: update install script, correct gazebo related model xacro files; transmission + models

File: urdf/ur5e_with_r85_mounting_structure.urdf.xacro (robot description, xacro)
@@ -34,6 +34,8 @@
     <xacro:include filename="$(find ur5e_workstation)/urdf/ur_e_transmission.xacro" />
     <xacro:include filename="$(find ur5e_workstation)/urdf/ur_e_gazebo.xacro" />
-    <xacro:ur_arm_transmission prefix="${prefix}" />
+    <xacro:include filename="$(find ur5e_workstation)/urdf/depth_camera_gazebo.xacro" />
+    <xacro:ur_arm_transmission prefix="${prefix}" namespace="ur5e" />
     <xacro:ur_arm_gazebo prefix="${prefix}" />
+    <xacro:ur_depth_gazebo prefix="${prefix}" />
     <!-- Inertia parameters -->
     <xacro:property name="base_mass" value="4.0" />  <!-- This mass might be incorrect -->
@@ -404,4 +406,5 @@
         <inertia ixx="0" ixy="0" ixz="0" iyy="0" iyz="0" izz="0" />
       </inertial>
+<!-- This is a dummy camera link used to properly avoid obstacles, does not need to be visualized
       <visual>
         <origin xyz="0 0 0" rpy="0 0 0" />
@@ -413,4 +416,5 @@
         </material>
       </visual>
+-->
       <collision>
         <origin xyz="0 0 0" rpy="0 0 0" />
@@ -426,4 +430,21 @@
       <axis xyz="0 0 0" />
     </joint>
+<!-- ########## Joints/links specifically for Gazebo simulated 2D and depth camera ########## -->
+    <!-- Create a virtual joint between d435 and gazebo camera link -->
+    <joint name="${prefix}d435_gazebo_camera_joint" type="fixed">
+      <origin xyz="0 0 0.013" rpy="-1.57 -1.57 0.0"/>
+      <parent link="${prefix}d435"/>
+      <child link="${prefix}gazebo_camera"/>
+    </joint>
+    <link name="${prefix}gazebo_camera" />
+    <!-- Create a virtual joint between d435_mount_link and gazebo depth camera link -->
+    <joint name="${prefix}d435_mount_to_gazebo_depth_camera_joint" type="fixed">
+      <origin xyz="0 -0.013 0.09" rpy="1.5708 3.1416 0" />
+      <parent link="${prefix}d435_mount_link" />
+      <child link="${prefix}gazebo_depth_camera" />
+      <axis xyz="0 0 0" />
+    </joint>
+    <link name="${prefix}gazebo_depth_camera" />
+<!-- ########## Joints/links specifically for Gazebo simulated 2D and depth camera ########## -->
     <link name="${prefix}millibar_adapters_link">
       <inertial>

File: urdf/ur_e_transmission.xacro (robot description, xacro)
@@ -13,8 +13,10 @@
     xmlns:physics="http://playerstage.sourceforge.net/gazebo/xmlschema/#physics"
     xmlns:xacro="http://ros.org/wiki/xacro" name="ur5e_d435_millibar_combined_r2f85" >
-  <xacro:macro name="ur_arm_transmission" params="prefix">
+  <xacro:macro name="ur_arm_transmission" params="prefix namespace">
     <gazebo>
       <plugin name="gazebo_ros_control" filename="libgazebo_ros_control.so">
-        <robotNamespace>/ur5e</robotNamespace>
+        <robotNamespace>/${namespace}</robotNamespace>
+        <robotSimType>gazebo_ros_control/DefaultRobotHWSim</robotSimType>
+        <legacyModeNS>true</legacyModeNS>
       </plugin>
     </gazebo>
